Commit message: sim progress

File: turtlebot3_simulations/turtlebot3_gazebo/urdf/turtlebot3_burger.urdf (robot description, URDF)
Before this commit: robot turtlebot3_burger, 9 links, 8 joints
Links:
- added link camera_link; visual box 
Joints:
- added joint camera_joint: type fixed, parent , child , axis 

File: turtlebot3_simulations/turtlebot3_gazebo/urdf/turtlebot3_velodyne_burger.urdf (robot description, URDF)
Before this commit: robot turtlebot3_burger, 9 links, 8 joints
Links:
- added link camera_link; visual box 
Joints:
- added joint camera_joint: type fixed, parent , child , axis 
